File: hw/sumobot/qrsumo.kicad_sch (KiCad schematic)
At the start: 76 parts, among them J1 Conn_01x02, J2 USB_B_Micro, J3 UART, J4 MOTOR_LEFT, J5 MOTOR_RIGHT, J6 Conn_01x07, J7 Conn_01x07, J8 VBAT, Q1 AO3400A, Q2 DMG2301L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

Commit message: Add schematic details
Other:
- company: (none) -> Qrtech
- title: (none) -> QRsumo
Changed lines of the file:
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@@
 (kicad_sch (version 20211123) (generator eeschema)
   (paper "A3")
+  (title_block
+    (title "QRsumo")
+    (date "2023-06-07")
+    (rev "1.0")
+    (company "Qrtech")
+  )
   (junction (at 42.545 53.34) (diameter 0) (color 0 0 0 0)
   )
